File: hw/air-stcc4/0.1.0/air-stcc4.kicad_pcb (KiCad board)
At the start: 2 copper layers, 25 x 20 mm, 16 parts, among them J1 BM04B-SRSS-TB(LF)(SN), J2 BM04B-SRSS-TB(LF)(SN), J3 Conn_01x05, M1 MountingHole_2.2mm_M2, M2 MountingHole_2.2mm_M2, M3 MountingHole_2.2mm_M2, M4 MountingHole_2.2mm_M2, U1 STCC4, U2 SHT40

Commit message: added CTRLH logo ; fixed MPN for 10K resistors
Parts:
- added REF**: CTRLH Logo, 1myFootprints:CTRLH Logo, B.Cu at (24.9, 33.0)
- added REF**: OSHW-Logo2_7.3x6mm_SilkScreen, Symbol:OSHW-Logo2_7.3x6mm_SilkScreen, B.Cu at (24.0, 26.0)

Commit message: doc improvements
fixed LED footprint on air-stcc4/0.1.0 (changed to 0603)
Parts:
- D1: footprint LED_SMD:LED_0201_0603Metric_Pad0.64x0.40mm_HandSolder -> LED_SMD:LED_0603_1608Metric_Pad1.05x0.95mm_HandSolder
- moved D1 0.50 mm to (30.0, 22.4)
Routing:
- net Net-(D1-A): track 1.60 -> 2.96 mm
- net GND: track 22.8 -> 23.8 mm
Other:
- board text added: "25mm x 20mm m.2 mounts 2.5mm offset"
